File: HS_MUX.kicad_sch (KiCad schematic)
At the start: 2 parts, among them U2 CBTL02043A, U3 TS3USB30EDGSR

Commit message: Weiter gearbeitet
Fast fertig:
HUB
Fertig
Connector (Up and Down)
MUX
Parts:
- added C15, C16: 100n, Capacitor_SMD:C_0402_1005Metric, symbol Device:C
- added R30: 10k, Resistor_SMD:R_0402_1005Metric, symbol Device:R
- added R31: 1k, Resistor_SMD:R_0402_1005Metric, symbol Device:R
Connections:
- net +3.3V: now also U2.1 (VDD), U2.10 (VDD), U2.6 (VDD), U3.10 (VCC), C15.2, C16.2, R31.1
- net GND: now also U2.11 (GND), U2.20 (GND), U2.21 (GND), U2.5 (GND), U3.5 (GND), C15.1, C16.1, R30.2
- net USB_UP2_SSTX_C_N: now reaches U2.12 (C1_N)
- net USB_UP2_SSTX_C_P: now reaches U2.13 (C1_P)
- net USB_UP2_SSRX_C_N: now reaches U2.14 (C0_N)
- net USB_UP2_SSRX_C_P: now reaches U2.15 (C0_P)
- net USB_UP1_SSTX_C_N: now reaches U2.16 (B1_N)
- net USB_UP1_SSTX_C_P: now reaches U2.17 (B1_P)
- net USB_UP1_SSRX_C_N: now reaches U2.18 (B0_N)
- net USB_UP1_SSRX_C_P: now reaches U2.19 (B0_P)
- net ~{MUX_OE}: now reaches U2.2 (XSD)
- net ~{MUX_OE}: now also U3.9 (~{OE}), R30.1, R31.2
- net USB_UPSW_SSRX_C_P: now reaches U2.3 (A0_P)
- net USB_UPSW_SSRX_C_N: now reaches U2.4 (A0_N)
- net USB_UPSW_SSTX_C_P: now reaches U2.7 (A1_P)
- net USB_UPSW_SSTX_C_N: now reaches U2.8 (A1_N)
- net DIRECTION_SELECT: now reaches U2.9 (SEL)
- net DIRECTION_SELECT: now also U3.1 (S)
- net USB_UP1_D_P: now reaches U3.2 (D1+)
- net USB_UP2_D_P: now reaches U3.3 (D2+)
- net USB_UPSW_D_P: now reaches U3.4 (D+)
- net USB_UPSW_D_N: now reaches U3.6 (D-)
- net USB_UP2_D_N: now reaches U3.7 (D2-)
- net USB_UP1_D_N: now reaches U3.8 (D1-)
Other:
- note added: "MUX Default ON"
- moved on the sheet: U2, U3

Commit message: Footprints Updated
Parts:
- C15, C16: footprint Capacitor_SMD:C_0402_1005Metric -> 00_Capacitor:Cap_0402
- R30, R31: footprint Resistor_SMD:R_0402_1005Metric -> 00_Resistor:Res_0402
Changed lines of the file:
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@@
 			)
 		)
-		(property "Footprint" "Resistor_SMD:R_0402_1005Metric"
+		(property "Footprint" "00_Resistor:Res_0402"
 			(at 238.252 29.21 90)
 			(effects
@@
 			)
 		)
-		(property "Footprint" "Capacitor_SMD:C_0402_1005Metric"
+		(property "Footprint" "00_Capacitor:Cap_0402"
 			(at 129.8448 153.67 0)
 			(effects
@@
 			)
 		)
-		(property "Footprint" "Resistor_SMD:R_0402_1005Metric"
+		(property "Footprint" "00_Resistor:Res_0402"
 			(at 238.252 39.37 90)
 			(effects
@@
 			)
 		)
-		(property "Footprint" "Capacitor_SMD:C_0402_1005Metric"
+		(property "Footprint" "00_Capacitor:Cap_0402"
 			(at 131.1148 26.67 0)
 			(effects

Commit message: USB 3 Stecker ausgetauscht
Parts:
- renumbered C16 to C41, C15 to C42, R31 to R25, R30 to R26, U2 to U4
Changed lines of the file:
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@@
 		(on_board yes)
 		(dnp no)
-		(property "Reference" "#PWR08"
+		(property "Reference" "#PWR054"
 			(at 132.08 52.07 0)
 			(effects
@@
 			(project ""
 				(path "/96aa4cdc-6548-43b6-b96a-6d1618c17d83/51eaf119-28f7-4fb3-b499-06b3f53ecd18"
-					(reference "#PWR08")
+					(reference "#PWR054")
 					(unit 1)
 				)
@@
 		(on_board yes)
 		(dnp no)
-		(property "Reference" "#PWR035"
+		(property "Reference" "#PWR050"
 			(at 130.81 156.21 0)
 			(effects
@@
 			(project "USB_3_SWITCHER"
 				(path "/96aa4cdc-6548-43b6-b96a-6d1618c17d83/51eaf119-28f7-4fb3-b499-06b3f53ecd18"
-					(reference "#PWR035")
+					(reference "#PWR050")
 					(unit 1)
 				)
@@
 		(on_board yes)
 		(dnp no)
-		(property "Reference" "#PWR065"
+		(property "Reference" "#PWR057"
 			(at 240.03 52.07 0)
 			(effects
@@
 			(project "USB_3_SWITCHER"
 				(path "/96aa4cdc-6548-43b6-b96a-6d1618c17d83/51eaf119-28f7-4fb3-b499-06b3f53ecd18"
-					(reference "#PWR065")
+					(reference "#PWR057")
 					(unit 1)
 				)
@@
 		(dnp no)
 		(fields_autoplaced yes)
-		(property "Reference" "U2"
+		(property "Reference" "U4"
 			(at 129.9367 48.26 0)
 			(effects
@@
 			(project "USB_3_SWITCHER"
 				(path "/96aa4cdc-6548-43b6-b96a-6d1618c17d83/51eaf119-28f7-4fb3-b499-06b3f53ecd18"
-					(reference "U2")
+					(reference "U4")
 					(unit 1)
 				)
@@
 		(on_board yes)
 		(dnp no)
-		(property "Reference" "#PWR011"
+		(property "Reference" "#PWR049"
 			(at 130.81 147.32 0)
 			(effects
@@
 			(project ""
 				(path "/96aa4cdc-6548-43b6-b96a-6d1618c17d83/51eaf119-28f7-4fb3-b499-06b3f53ecd18"
-					(reference "#PWR011")
+					(reference "#PWR049")
 					(unit 1)
 				)
@@
 		(on_board yes)
 		(dnp no)
-		(property "Reference" "#PWR036"
+		(property "Reference" "#PWR051"
 			(at 130.81 168.91 0)
 			(effects
@@
 			(project "USB_3_SWITCHER"
 				(path "/96aa4cdc-6548-43b6-b96a-6d1618c17d83/51eaf119-28f7-4fb3-b499-06b3f53ecd18"
-					(reference "#PWR036")
+					(reference "#PWR051")
 					(unit 1)
 				)
@@
 		(dnp yes)
 		(fields_autoplaced yes)
-		(property "Reference" "R31"
+		(property "Reference" "R25"
 			(at 242.57 27.9399 0)
 			(effects
@@
 			(project "USB_3_SWITCHER"
 				(path "/96aa4cdc-6548-43b6-b96a-6d1618c17d83/51eaf119-28f7-4fb3-b499-06b3f53ecd18"
-					(reference "R31")
+					(reference "R25")
 					(unit 1)
 				)
@@
 		(on_board yes)
 		(dnp no)
-		(property "Reference" "#PWR09"
+		(property "Reference" "#PWR048"
 			(at 130.81 119.38 0)
 			(effects
@@
 			(project ""
 				(path "/96aa4cdc-6548-43b6-b96a-6d1618c17d83/51eaf119-28f7-4fb3-b499-06b3f53ecd18"
-					(reference "#PWR09")
+					(reference "#PWR048")
 					(unit 1)
 				)
@@
 		(on_board yes)
 		(dnp no)
-		(property "Reference" "#PWR034"
+		(property "Reference" "#PWR053"
 			(at 132.08 41.91 0)
 			(effects
@@
 			(project "USB_3_SWITCHER"
 				(path "/96aa4cdc-6548-43b6-b96a-6d1618c17d83/51eaf119-28f7-4fb3-b499-06b3f53ecd18"
-					(reference "#PWR034")
+					(reference "#PWR053")
 					(unit 1)
 				)
@@
 		(on_board yes)
 		(dnp no)
-		(property "Reference" "C16"
+		(property "Reference" "C41"
 			(at 134.62 156.2099 0)
 			(effects
@@
 			(project "USB_3_SWITCHER"
 				(path "/96aa4cdc-6548-43b6-b96a-6d1618c17d83/51eaf119-28f7-4fb3-b499-06b3f53ecd18"
-					(reference "C16")
+					(reference "C41")
 					(unit 1)
 				)
@@
 		(dnp no)
 		(fields_autoplaced yes)
-		(property "Reference" "R30"
+		(property "Reference" "R26"
 			(at 242.57 38.0999 0)
 			(effects
@@
 			(project "USB_3_SWITCHER"
 				(path "/96aa4cdc-6548-43b6-b96a-6d1618c17d83/51eaf119-28f7-4fb3-b499-06b3f53ecd18"
-					(reference "R30")
+					(reference "R26")
 					(unit 1)
 				)
@@
 		(on_board yes)
 		(dnp no)
-		(property "Reference" "C15"
+		(property "Reference" "C42"
 			(at 135.89 29.2099 0)
 			(effects
@@
 			(project "USB_3_SWITCHER"
 				(path "/96aa4cdc-6548-43b6-b96a-6d1618c17d83/51eaf119-28f7-4fb3-b499-06b3f53ecd18"
-					(reference "C15")
+					(reference "C42")
 					(unit 1)
 				)
@@
 		(on_board yes)
 		(dnp no)
-		(property "Reference" "#PWR067"
+		(property "Reference" "#PWR056"
 			(at 240.03 27.94 0)
 			(effects
@@
 			(project "USB_3_SWITCHER"
 				(path "/96aa4cdc-6548-43b6-b96a-6d1618c17d83/51eaf119-28f7-4fb3-b499-06b3f53ecd18"
-					(reference "#PWR067")
+					(reference "#PWR056")
 					(unit 1)
 				)
@@
 		(on_board yes)
 		(dnp no)
-		(property "Reference" "#PWR033"
+		(property "Reference" "#PWR052"
 			(at 132.08 29.21 0)
 			(effects
@@
 			(project "USB_3_SWITCHER"
 				(path "/96aa4cdc-6548-43b6-b96a-6d1618c17d83/51eaf119-28f7-4fb3-b499-06b3f53ecd18"
-					(reference "#PWR033")
+					(reference "#PWR052")
 					(unit 1)
 				)
@@
 		(on_board yes)
 		(dnp no)
-		(property "Reference" "#PWR010"
+		(property "Reference" "#PWR055"
 			(at 132.08 105.41 0)
 			(effects
@@
 			(project ""
 				(path "/96aa4cdc-6548-43b6-b96a-6d1618c17d83/51eaf119-28f7-4fb3-b499-06b3f53ecd18"
-					(reference "#PWR010")
-					(unit 1)
-				)
+					(reference "#PWR055")
+					(unit 1)
+				)

Commit message: Weiter gemacht
Parts:
- added C20: 100n, 00_Capacitor:Cap_0402, symbol Device:C
Connections:
- net +3.3V: now also C20.2
- net GND: now also C20.1
Other:
- moved on the sheet: C42

Commit message: weiter gemacht
Connections:
- net USB_UP2_SSTX_C_N: now also U4.13 (C1_P); no longer U4.12 (C1_N)
- net USB_UP2_SSTX_C_P: now also U4.12 (C1_N); no longer U4.13 (C1_P)

Commit message: Weiter gemacht
Connections:
- net USB_UP2_SSTX_C_N: now also U4.12 (C1_N); no longer U4.13 (C1_P)
- net USB_UP2_SSTX_C_P: now also U4.13 (C1_P); no longer U4.12 (C1_N)
Changed lines of the file:
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@@
 		)
 	)
-	(hierarchical_label "USB_UP2_SSTX_C_N"
+	(hierarchical_label "USB_UP2_SSTX_C_P"
 		(shape output)
 		(at 69.85 76.2 180)
@@
 		)
 	)
-	(hierarchical_label "USB_UP2_SSTX_C_P"
+	(hierarchical_label "USB_UP2_SSTX_C_N"
 		(shape output)
 		(at 69.85 78.74 180)

Commit message: Layout + Schematic weiter gemacht
Parts:
- added C108: 100n, 00_Capacitor:Cap_0402, symbol Device:C
- U3: footprint Package_SO:VSSOP-10_3x3mm_P0.5mm -> Package_SO:HVSSOP-10-1EP_3x3mm_P0.5mm_EP1.83x1.89mm
Connections:
- net +3.3V: now also C108.2
- net GND: now also C108.1
