File: USB_3_SWITCHER.kicad_pcb (KiCad board)
At the start: 2 copper layers, 170 parts, among them J2 Wuerth_USB3_B_Receptable_6922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, J3 Wuerth_USB3_B_Receptable_6922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, J4 Wuerth_USB3_Receptible_692122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, J5 Wuerth_USB3_Receptible_692122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, J6 Wuerth_USB3_Receptible_692122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, J7 Wuerth_USB3_Receptible_692122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, U1 AT24CS04-SSHM, U10 LM66100DCK, U11 TPD6E05U06RVZ, U12 MAX8586, U13 TPD6E05U06RVZ, U14 MAX8586, U15 TPD6E05U06RVZ, U16 MAX8586, U17 TPD6E05U06RVZ, U18 MAX8586, U19 TPD6E05U06RVZ, U2 TUSB8043A, U3 TS3USB30EDGSR, U4 CBTL02043A, U5 LM66100DCK, U6 LMR33640ADDA, U7 LMR33640ADDA, U8 LM66100DCK, U9 TPD6E05U06RVZ

Commit message: Weiter gemacht
Parts:
- removed C21, C22, C23, C24, C25, C26, C27, C28, C29, C30, C31, C32, C33, C34, C35: 100n, 00_Capacitor:Cap_0402
- added C100: 220n, 00_Capacitor:Cap_0402, F.Cu at (243.5, 132.9)
- added C101: 1u, 00_Capacitor:Cap_0402, F.Cu at (252.3, 136.3)
- added C102: 100n, 00_Capacitor:Cap_0402, F.Cu at (252.6, 134.0)
- added C103: 22u, 00_Capacitor:Cap_0805, F.Cu at (249.4, 129.5)
- added C104: 22u, 00_Capacitor:Cap_0805, F.Cu at (249.4, 127.7)
- added C105: 22u, 00_Capacitor:Cap_0805, F.Cu at (249.4, 125.9)
- added C87: 10u, 00_Capacitor:Cap_0603, F.Cu at (229.9, 143.2)
- added C88: 10u, 00_Capacitor:Cap_0603, F.Cu at (230.0, 142.0)
- added C89: 22u, 00_Capacitor:Cap_0805, F.Cu at (249.8, 143.3)
- added C90: 100uF, Capacitor_SMD:CP_Elec_6.3x5.9, F.Cu at (236.4, 135.2)
- added C91: 100n, 00_Capacitor:Cap_0402, F.Cu at (253.1, 148.1)
- added C92: 22u, 00_Capacitor:Cap_0805, F.Cu at (249.8, 141.6)
- added C93: 22u, 00_Capacitor:Cap_0805, F.Cu at (249.8, 139.9)
- added C94: 10u, 00_Capacitor:Cap_0603, F.Cu at (242.6, 147.1)
- added C95: 220n, 00_Capacitor:Cap_0402, F.Cu at (243.8, 147.1)
- added C96: 10u, 00_Capacitor:Cap_0603, F.Cu at (218.5, 141.9)
- added C97: 10u, 00_Capacitor:Cap_0603, F.Cu at (182.2, 141.9)
- added C98: 1u, 00_Capacitor:Cap_0402, F.Cu at (252.6, 149.7)
- added C99: 10u, 00_Capacitor:Cap_0603, F.Cu at (242.4, 133.0)
- added D1: D_Schottky, Diode_SMD:D_SOD-323, F.Cu at (216.0, 143.6)
- added D2: D_Schottky, Diode_SMD:D_SOD-323, F.Cu at (179.8, 143.6)
- added H1: MountingHole_Pad_MP, MountingHole:MountingHole_3.2mm_M3_DIN965_Pad_TopBottom, F.Cu at (258.4, 107.2)
- added H2: MountingHole_Pad_MP, MountingHole:MountingHole_3.2mm_M3_DIN965_Pad_TopBottom, F.Cu at (145.9, 107.2)
- added H3: MountingHole_Pad_MP, MountingHole:MountingHole_3.2mm_M3_DIN965_Pad_TopBottom, F.Cu at (258.0, 154.0)
- added H4: MountingHole_Pad_MP, MountingHole:MountingHole_3.2mm_M3_DIN965_Pad_TopBottom, F.Cu at (146.4, 154.0)
- added J1: Jack-DC, Connector_BarrelJack:BarrelJack_GCT_DCJ200-10-A_Horizontal, F.Cu at (232.4, 149.2)
- added J8: Conn_01x16_MountingPin, Connector_PinHeader_2.54mm:PinHeader_2x08_P2.54mm_Vertical_SMD, F.Cu at (194.4, 147.2)
- added J9: Conn_01x04_MountingPin, Connector_PinHeader_2.54mm:PinHeader_1x04_P2.54mm_Vertical_SMD_Pin1Left, F.Cu at (156.1, 152.0)
- added L1: 6.8u, Inductor_SMD:L_Coilcraft_XAL7030-272, F.Cu at (256.4, 143.2)
- added L2: 10u, Inductor_SMD:L_Coilcraft_XAL7030-272, F.Cu at (255.9, 129.2)
- added R56: 100k, 00_Capacitor:Cap_0402, B.Cu at (250.9, 149.4)
- added R57: 4.32k, 00_Capacitor:Cap_0402, B.Cu at (250.9, 151.1)
- added R58: 100k, 00_Capacitor:Cap_0402, B.Cu at (250.6, 135.2)
- added R59: 1K, 00_Capacitor:Cap_0402, B.Cu at (250.6, 136.9)
- added Y1: 24MHz 20ppm, Crystal:Crystal_SMD_3225-4Pin_3.2x2.5mm, F.Cu at (162.7, 144.2)
- C10, C11, C12, C13, C15, C16, C17, C18, C19, C36, C37, C38, C39, C40, C42, C43, C6, C63, C64, C65, C70, C71, C72, C77, C78, C79, C84, C85, C86, C9, FB1, FB2, FB3, FB4, R27, R28, R36, R37, R38, R39, R40, R41, R42, R43, R44, R45, R46, R47, R48, R49, R50, R51, R52, R53, R54, R55, U12, U14, U16, U18: moved to B.Cu
- moved J4 175.5 mm to (241.8, 104.2), turned to 180 degrees
- moved R38 171.7 mm to (249.7, 115.7), turned to 90 degrees
- moved R39 170.3 mm to (248.5, 118.8), turned to 90 degrees
- moved R40 169.9 mm to (247.7, 118.8), turned to -90 degrees
- moved R37 167.9 mm to (246.9, 118.8), turned to -90 degrees
- moved R36 166.7 mm to (246.1, 118.8), turned to -90 degrees
- moved C63 165.5 mm to (245.3, 116.7), turned to -90 degrees
- moved FB1 165.2 mm to (245.5, 111.9), turned to -90 degrees
- moved U12 164.9 mm to (247.5, 115.8), turned to 90 degrees
- moved C64 164.2 mm to (247.2, 111.8), turned to 90 degrees
- moved C62 161.9 mm to (243.4, 122.3), turned to 90 degrees
- moved C65 161.5 mm to (243.9, 111.8), turned to 90 degrees
- moved U13 161.3 mm to (241.8, 119.2), turned to 90 degrees
- moved C60 160.4 mm to (242.7, 122.3), turned to 90 degrees
- moved C61 159.1 mm to (240.9, 122.2), turned to 90 degrees
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Connections:
- C20 pad 1: /DOWNSTREAM_CONNECTORS/USB_DS_SSTX_C_N -> GND
- C20 pad 2: /USB_HUB/USB_DS1_SSTX_N -> +3.3V
- U11 pad 1: /UPSTREAM_CON1/USB_UP_D_N -> /UPSTREAM_CON1/USB_UP_SSRX_N
- U11 pad 11: /UPSTREAM_CON1/USB_UP_SSRX_P -> /UPSTREAM_CON1/USB_UP_D_P
- U11 pad 12: /UPSTREAM_CON1/USB_UP_SSRX_N -> /UPSTREAM_CON1/USB_UP_D_N
- U11 pad 13: /UPSTREAM_CON1/USB_UP_D_P -> /UPSTREAM_CON1/USB_UP_SSRX_P
- U11 pad 14: /UPSTREAM_CON1/USB_UP_D_N -> /UPSTREAM_CON1/USB_UP_SSRX_N
- U11 pad 2: /UPSTREAM_CON1/USB_UP_D_P -> /UPSTREAM_CON1/USB_UP_SSRX_P
- U11 pad 3: /UPSTREAM_CON1/USB_UP_SSRX_N -> /UPSTREAM_CON1/USB_UP_D_N
- U11 pad 4: /UPSTREAM_CON1/USB_UP_SSRX_P -> /UPSTREAM_CON1/USB_UP_D_P
- U11 pad 6: /UPSTREAM_CON1/USB_UP_SSTX_N -> /UPSTREAM_CON1/USB_UP_SSTX_P
- U11 pad 7: /UPSTREAM_CON1/USB_UP_SSTX_P -> /UPSTREAM_CON1/USB_UP_SSTX_N
- U11 pad 8: /UPSTREAM_CON1/USB_UP_SSTX_P -> /UPSTREAM_CON1/USB_UP_SSTX_N
- U11 pad 9: /UPSTREAM_CON1/USB_UP_SSTX_N -> /UPSTREAM_CON1/USB_UP_SSTX_P
- U13 pad 1: /DOWNSTREAM_CONNECTORS/USB_DS_D_N -> /DOWNSTREAM_CONNECTORS/USB_DS_SSRX_N
- U13 pad 11: /DOWNSTREAM_CONNECTORS/USB_DS_SSRX_P -> /DOWNSTREAM_CONNECTORS/USB_DS_D_N
- U13 pad 12: /DOWNSTREAM_CONNECTORS/USB_DS_SSRX_N -> /DOWNSTREAM_CONNECTORS/USB_DS_D_P
- U13 pad 13: /DOWNSTREAM_CONNECTORS/USB_DS_D_P -> /DOWNSTREAM_CONNECTORS/USB_DS_SSRX_P
- U13 pad 14: /DOWNSTREAM_CONNECTORS/USB_DS_D_N -> /DOWNSTREAM_CONNECTORS/USB_DS_SSRX_N
- U13 pad 2: /DOWNSTREAM_CONNECTORS/USB_DS_D_P -> /DOWNSTREAM_CONNECTORS/USB_DS_SSRX_P
- U13 pad 3: /DOWNSTREAM_CONNECTORS/USB_DS_SSRX_N -> /DOWNSTREAM_CONNECTORS/USB_DS_D_P
- U13 pad 4: /DOWNSTREAM_CONNECTORS/USB_DS_SSRX_P -> /DOWNSTREAM_CONNECTORS/USB_DS_D_N
- U15 pad 1: /DOWNSTREAM_CONNECTORS1/USB_DS_D_N -> /DOWNSTREAM_CONNECTORS1/USB_DS_SSRX_N
- U15 pad 11: /DOWNSTREAM_CONNECTORS1/USB_DS_SSRX_P -> /DOWNSTREAM_CONNECTORS1/USB_DS_D_N
- U15 pad 12: /DOWNSTREAM_CONNECTORS1/USB_DS_SSRX_N -> /DOWNSTREAM_CONNECTORS1/USB_DS_D_P
- U15 pad 13: /DOWNSTREAM_CONNECTORS1/USB_DS_D_P -> /DOWNSTREAM_CONNECTORS1/USB_DS_SSRX_P
- U15 pad 14: /DOWNSTREAM_CONNECTORS1/USB_DS_D_N -> /DOWNSTREAM_CONNECTORS1/USB_DS_SSRX_N
- U15 pad 2: /DOWNSTREAM_CONNECTORS1/USB_DS_D_P -> /DOWNSTREAM_CONNECTORS1/USB_DS_SSRX_P
- U15 pad 3: /DOWNSTREAM_CONNECTORS1/USB_DS_SSRX_N -> /DOWNSTREAM_CONNECTORS1/USB_DS_D_P
- U15 pad 4: /DOWNSTREAM_CONNECTORS1/USB_DS_SSRX_P -> /DOWNSTREAM_CONNECTORS1/USB_DS_D_N
- U17 pad 1: /DOWNSTREAM_CONNECTORS2/USB_DS_D_N -> /DOWNSTREAM_CONNECTORS2/USB_DS_SSRX_N
- U17 pad 11: /DOWNSTREAM_CONNECTORS2/USB_DS_SSRX_P -> /DOWNSTREAM_CONNECTORS2/USB_DS_D_N
- U17 pad 12: /DOWNSTREAM_CONNECTORS2/USB_DS_SSRX_N -> /DOWNSTREAM_CONNECTORS2/USB_DS_D_P
- U17 pad 13: /DOWNSTREAM_CONNECTORS2/USB_DS_D_P -> /DOWNSTREAM_CONNECTORS2/USB_DS_SSRX_P
- U17 pad 14: /DOWNSTREAM_CONNECTORS2/USB_DS_D_N -> /DOWNSTREAM_CONNECTORS2/USB_DS_SSRX_N
- U17 pad 2: /DOWNSTREAM_CONNECTORS2/USB_DS_D_P -> /DOWNSTREAM_CONNECTORS2/USB_DS_SSRX_P
- U17 pad 3: /DOWNSTREAM_CONNECTORS2/USB_DS_SSRX_N -> /DOWNSTREAM_CONNECTORS2/USB_DS_D_P
- U17 pad 4: /DOWNSTREAM_CONNECTORS2/USB_DS_SSRX_P -> /DOWNSTREAM_CONNECTORS2/USB_DS_D_N
- U19 pad 1: /DOWNSTREAM_CONNECTORS3/USB_DS_D_N -> /DOWNSTREAM_CONNECTORS3/USB_DS_SSRX_N
- U19 pad 11: /DOWNSTREAM_CONNECTORS3/USB_DS_SSRX_P -> /DOWNSTREAM_CONNECTORS3/USB_DS_D_N
- U19 pad 12: /DOWNSTREAM_CONNECTORS3/USB_DS_SSRX_N -> /DOWNSTREAM_CONNECTORS3/USB_DS_D_P
- U19 pad 13: /DOWNSTREAM_CONNECTORS3/USB_DS_D_P -> /DOWNSTREAM_CONNECTORS3/USB_DS_SSRX_P
- U19 pad 14: /DOWNSTREAM_CONNECTORS3/USB_DS_D_N -> /DOWNSTREAM_CONNECTORS3/USB_DS_SSRX_N
- U19 pad 2: /DOWNSTREAM_CONNECTORS3/USB_DS_D_P -> /DOWNSTREAM_CONNECTORS3/USB_DS_SSRX_P
- U19 pad 3: /DOWNSTREAM_CONNECTORS3/USB_DS_SSRX_N -> /DOWNSTREAM_CONNECTORS3/USB_DS_D_P
- U19 pad 4: /DOWNSTREAM_CONNECTORS3/USB_DS_SSRX_P -> /DOWNSTREAM_CONNECTORS3/USB_DS_D_N
- U2 pad 11: /USB_HUB/USB_DS2_SSTX_P -> /DOWNSTREAM_CONNECTORS1/USB_DS_SSTX_C_P
- U2 pad 12: /USB_HUB/USB_DS2_SSTX_N -> /DOWNSTREAM_CONNECTORS1/USB_DS_SSTX_C_N
- U2 pad 14: /USB_HUB/USB_DS2_SSRX_P -> /DOWNSTREAM_CONNECTORS1/USB_DS_SSRX_C_P
- U2 pad 15: /USB_HUB/USB_DS2_SSRX_N -> /DOWNSTREAM_CONNECTORS1/USB_DS_SSRX_C_N
- U2 pad 19: /USB_HUB/USB_DS3_SSTX_P -> /DOWNSTREAM_CONNECTORS2/USB_DS_SSTX_C_P
- U2 pad 20: /USB_HUB/USB_DS3_SSTX_N -> /DOWNSTREAM_CONNECTORS2/USB_DS_SSTX_C_N
- U2 pad 22: /USB_HUB/USB_DS3_SSRX_P -> /DOWNSTREAM_CONNECTORS2/USB_DS_SSRX_C_P
- U2 pad 23: /USB_HUB/USB_DS3_SSRX_N -> /DOWNSTREAM_CONNECTORS2/USB_DS_SSRX_C_N
- U2 pad 26: /USB_HUB/USB_DS4_SSTX_P -> /DOWNSTREAM_CONNECTORS3/USB_DS_SSTX_C_P
- U2 pad 27: /USB_HUB/USB_DS4_SSTX_N -> /DOWNSTREAM_CONNECTORS3/USB_DS_SSTX_C_N
- U2 pad 29: /USB_HUB/USB_DS4_SSRX_P -> /DOWNSTREAM_CONNECTORS3/USB_DS_SSRX_C_P
- U2 pad 3: /USB_HUB/USB_DS1_SSTX_P -> /DOWNSTREAM_CONNECTORS/USB_DS_SSTX_C_P
- U2 pad 30: /USB_HUB/USB_DS4_SSRX_N -> /DOWNSTREAM_CONNECTORS3/USB_DS_SSRX_C_N
- U2 pad 4: /USB_HUB/USB_DS1_SSTX_N -> /DOWNSTREAM_CONNECTORS/USB_DS_SSTX_C_N
- U2 pad 6: /USB_HUB/USB_DS1_SSRX_P -> /DOWNSTREAM_CONNECTORS/USB_DS_SSRX_C_P
- U2 pad 7: /USB_HUB/USB_DS1_SSRX_N -> /DOWNSTREAM_CONNECTORS/USB_DS_SSRX_C_N
- U6 pad 1: Net-(U6-GND-Pad1) -> GND
- U6 pad 2: unconnected-(U6-VIN-Pad2) -> +5V
- U6 pad 3: unconnected-(U6-EN-Pad3) -> /POWER_SUPPLY/BUCK_3V3_EN
- U6 pad 4: unconnected-(U6-PG-Pad4) -> /POWER_SUPPLY/BUCK_3V3_PG
- U6 pad 5: unconnected-(U6-FB-Pad5) -> /POWER_SUPPLY/BUCK_3V3_FB
- U6 pad 6: unconnected-(U6-VCC-Pad6) -> /POWER_SUPPLY/BUCK_3V3_VCC
- U6 pad 7: unconnected-(U6-BOOT-Pad7) -> Net-(U6-BOOT)
- U6 pad 8: unconnected-(U6-SW-Pad8) -> /POWER_SUPPLY/LX_3V3
- U6 pad 9: Net-(U6-GND-Pad1) -> GND
- U7 pad 1: Net-(U7-GND-Pad1) -> GND
- U7 pad 2: unconnected-(U7-VIN-Pad2) -> +5V
- U7 pad 3: unconnected-(U7-EN-Pad3) -> /POWER_SUPPLY/BUCK_1V1_EN
- U7 pad 4: unconnected-(U7-PG-Pad4) -> /POWER_SUPPLY/BUCK_1V1_PG
- U7 pad 5: unconnected-(U7-FB-Pad5) -> /POWER_SUPPLY/BUCK_1V1_FB
- U7 pad 6: unconnected-(U7-VCC-Pad6) -> /POWER_SUPPLY/BUCK_1V1_VCC
- U7 pad 7: unconnected-(U7-BOOT-Pad7) -> Net-(U7-BOOT)
- U7 pad 8: unconnected-(U7-SW-Pad8) -> /POWER_SUPPLY/LX_1V1
- U7 pad 9: Net-(U7-GND-Pad1) -> GND
- U9 pad 1: /UPSTREAM_CON/USB_UP_D_N -> /UPSTREAM_CON/USB_UP_SSRX_N
- U9 pad 11: /UPSTREAM_CON/USB_UP_SSRX_P -> /UPSTREAM_CON/USB_UP_D_P
- U9 pad 12: /UPSTREAM_CON/USB_UP_SSRX_N -> /UPSTREAM_CON/USB_UP_D_N
- U9 pad 13: /UPSTREAM_CON/USB_UP_D_P -> /UPSTREAM_CON/USB_UP_SSRX_P
- U9 pad 14: /UPSTREAM_CON/USB_UP_D_N -> /UPSTREAM_CON/USB_UP_SSRX_N
- U9 pad 2: /UPSTREAM_CON/USB_UP_D_P -> /UPSTREAM_CON/USB_UP_SSRX_P
- U9 pad 3: /UPSTREAM_CON/USB_UP_SSRX_N -> /UPSTREAM_CON/USB_UP_D_N
- U9 pad 4: /UPSTREAM_CON/USB_UP_SSRX_P -> /UPSTREAM_CON/USB_UP_D_P
- U9 pad 6: /UPSTREAM_CON/USB_UP_SSTX_N -> /UPSTREAM_CON/USB_UP_SSTX_P
- U9 pad 7: /UPSTREAM_CON/USB_UP_SSTX_P -> /UPSTREAM_CON/USB_UP_SSTX_N
- U9 pad 8: /UPSTREAM_CON/USB_UP_SSTX_P -> /UPSTREAM_CON/USB_UP_SSTX_N
- U9 pad 9: /UPSTREAM_CON/USB_UP_SSTX_N -> /UPSTREAM_CON/USB_UP_SSTX_P
Routing:
- net /DOWNSTREAM_CONNECTORS2/USB_DS_SSTX_C_N: track 0.00 -> 33.8 mm
- net /DOWNSTREAM_CONNECTORS2/USB_DS_SSTX_C_P: track 0.00 -> 33.8 mm
- net /DOWNSTREAM_CONNECTORS2/USB_DS_SSRX_C_P: track 0.00 -> 32.9 mm
- net /DOWNSTREAM_CONNECTORS2/USB_DS_SSRX_C_N: track 0.00 -> 32.9 mm
- net /UPSTREAM_CON1/USB_UP_D_P: track 0.00 -> 11.6 mm
- net /UPSTREAM_CON/USB_UP_D_P: track 0.00 -> 11.6 mm
- net /DOWNSTREAM_CONNECTORS3/USB_DS_SSTX_C_P: track 0.00 -> 11.3 mm
- net /DOWNSTREAM_CONNECTORS3/USB_DS_SSTX_C_N: track 0.00 -> 11.3 mm
- net /UPSTREAM_CON1/USB_UP_D_N: track 0.00 -> 11.2 mm
- net /UPSTREAM_CON/USB_UP_D_N: track 0.00 -> 11.2 mm
- net /DOWNSTREAM_CONNECTORS1/USB_DS_SSRX_P: track 0.00 -> 11.2 mm
- net /DOWNSTREAM_CONNECTORS2/USB_DS_SSRX_P: track 0.00 -> 11.2 mm
- net /DOWNSTREAM_CONNECTORS3/USB_DS_SSRX_P: track 0.00 -> 11.2 mm
- net /DOWNSTREAM_CONNECTORS/USB_DS_SSRX_P: track 0.00 -> 11.2 mm
- net /DOWNSTREAM_CONNECTORS2/USB_DS_SSRX_N: track 0.00 -> 11.2 mm
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Other:
- board outline added: 122 x 56 mm
- copper layers 2 -> 6

Commit message: weiter gemacht
Parts:
- H2: footprint MountingHole:MountingHole_3.2mm_M3_DIN965_Pad_TopBottom -> MountingHole:MountingHole_3.2mm_M3_Pad_TopBottom
- moved C42 2.51 mm to (204.9, 131.9)
- moved U3 2.50 mm to (204.8, 131.9)
- moved R26 2.20 mm to (195.2, 130.7)
- moved R25 2.20 mm to (195.2, 132.4)
- moved C3 1.04 mm to (164.6, 129.5)
- moved U4 0.25 mm to (190.5, 132.5)
Connections:
- C48 pad 1: /UPSTREAM_CON/USB_UP_SSRX_N -> /UPSTREAM_CON/USB_UP_SSRX_P
- C48 pad 2: /HS_MUX/USB_UP1_SSRX_C_N -> /HS_MUX/USB_UP1_SSRX_C_P
- C51 pad 1: /UPSTREAM_CON/USB_UP_SSRX_P -> /UPSTREAM_CON/USB_UP_SSRX_N
- C51 pad 2: /HS_MUX/USB_UP1_SSRX_C_P -> /HS_MUX/USB_UP1_SSRX_C_N
- C55 pad 1: /UPSTREAM_CON1/USB_UP_SSRX_N -> /UPSTREAM_CON1/USB_UP_SSRX_P
- C55 pad 2: /HS_MUX/USB_UP2_SSRX_C_N -> /HS_MUX/USB_UP2_SSRX_C_P
- C58 pad 1: /UPSTREAM_CON1/USB_UP_SSRX_P -> /UPSTREAM_CON1/USB_UP_SSRX_N
- C58 pad 2: /HS_MUX/USB_UP2_SSRX_C_P -> /HS_MUX/USB_UP2_SSRX_C_N
- J2 pad 8: /UPSTREAM_CON/USB_UP_SSRX_P -> /UPSTREAM_CON/USB_UP_SSRX_N
- J2 pad 9: /UPSTREAM_CON/USB_UP_SSRX_N -> /UPSTREAM_CON/USB_UP_SSRX_P
- J3 pad 8: /UPSTREAM_CON1/USB_UP_SSRX_P -> /UPSTREAM_CON1/USB_UP_SSRX_N
- J3 pad 9: /UPSTREAM_CON1/USB_UP_SSRX_N -> /UPSTREAM_CON1/USB_UP_SSRX_P
- U11 pad 1: /UPSTREAM_CON1/USB_UP_SSRX_N -> /UPSTREAM_CON1/USB_UP_SSRX_P
- U11 pad 13: /UPSTREAM_CON1/USB_UP_SSRX_P -> /UPSTREAM_CON1/USB_UP_SSRX_N
- U11 pad 14: /UPSTREAM_CON1/USB_UP_SSRX_N -> /UPSTREAM_CON1/USB_UP_SSRX_P
- U11 pad 2: /UPSTREAM_CON1/USB_UP_SSRX_P -> /UPSTREAM_CON1/USB_UP_SSRX_N
- U11 pad 6: /UPSTREAM_CON1/USB_UP_SSTX_P -> /UPSTREAM_CON1/USB_UP_SSTX_N
- U11 pad 7: /UPSTREAM_CON1/USB_UP_SSTX_N -> /UPSTREAM_CON1/USB_UP_SSTX_P
- U11 pad 8: /UPSTREAM_CON1/USB_UP_SSTX_N -> /UPSTREAM_CON1/USB_UP_SSTX_P
- U11 pad 9: /UPSTREAM_CON1/USB_UP_SSTX_P -> /UPSTREAM_CON1/USB_UP_SSTX_N
- U4 pad 12: /HS_MUX/USB_UP2_SSTX_C_N -> /HS_MUX/USB_UP2_SSTX_C_P
- U4 pad 13: /HS_MUX/USB_UP2_SSTX_C_P -> /HS_MUX/USB_UP2_SSTX_C_N
- U9 pad 1: /UPSTREAM_CON/USB_UP_SSRX_N -> /UPSTREAM_CON/USB_UP_SSRX_P
- U9 pad 13: /UPSTREAM_CON/USB_UP_SSRX_P -> /UPSTREAM_CON/USB_UP_SSRX_N
- U9 pad 14: /UPSTREAM_CON/USB_UP_SSRX_N -> /UPSTREAM_CON/USB_UP_SSRX_P
- U9 pad 2: /UPSTREAM_CON/USB_UP_SSRX_P -> /UPSTREAM_CON/USB_UP_SSRX_N
- U9 pad 6: /UPSTREAM_CON/USB_UP_SSTX_P -> /UPSTREAM_CON/USB_UP_SSTX_N
- U9 pad 7: /UPSTREAM_CON/USB_UP_SSTX_N -> /UPSTREAM_CON/USB_UP_SSTX_P
- U9 pad 8: /UPSTREAM_CON/USB_UP_SSTX_N -> /UPSTREAM_CON/USB_UP_SSTX_P
- U9 pad 9: /UPSTREAM_CON/USB_UP_SSTX_P -> /UPSTREAM_CON/USB_UP_SSTX_N
Routing:
- net /DOWNSTREAM_CONNECTORS/USB_DS_SSTX_C_P: track 2.65 -> 88.4 mm
- net /DOWNSTREAM_CONNECTORS/USB_DS_SSTX_C_N: track 2.65 -> 88.1 mm
- net /DOWNSTREAM_CONNECTORS/USB_DS_SSRX_C_P: track 5.28 -> 84.9 mm
- net /DOWNSTREAM_CONNECTORS/USB_DS_SSRX_C_N: track 5.09 -> 84.5 mm
- net /DOWNSTREAM_CONNECTORS1/USB_DS_SSTX_C_P: track 2.65 -> 59.0 mm
- net /DOWNSTREAM_CONNECTORS1/USB_DS_SSTX_C_N: track 2.65 -> 58.7 mm
- net /DOWNSTREAM_CONNECTORS1/USB_DS_SSRX_C_P: track 2.66 -> 55.8 mm
- net /DOWNSTREAM_CONNECTORS1/USB_DS_SSRX_C_N: track 2.66 -> 55.4 mm
- net /HS_MUX/USB_UP1_SSRX_C_N: track 0.00 -> 25.0 mm
- net /HS_MUX/USB_UP1_SSRX_C_P: track 0.00 -> 25.0 mm
- net /HS_MUX/USB_UP1_SSTX_C_N: track 0.00 -> 22.8 mm
- net /HS_MUX/USB_UP1_SSTX_C_P: track 0.00 -> 22.8 mm
- net /HS_MUX/USB_UP2_SSTX_C_P: track 0.00 -> 21.7 mm
- net /HS_MUX/USB_UP2_SSTX_C_N: track 0.00 -> 21.7 mm
- net /HS_MUX/USB_UP2_SSRX_C_N: track 0.00 -> 19.9 mm
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
Commit message: Weiter gemacht
Parts:
- removed C11: 100n, 00_Capacitor:Cap_0402
- C14, R1, R7: moved to B.Cu
- C42: moved to F.Cu
- moved L2 20.2 mm to (236.1, 133.2), turned to -90 degrees
- moved R16 17.0 mm to (142.6, 132.1), turned to 90 degrees
- moved C101 16.2 mm to (239.7, 126.1), turned to -90 degrees
- moved R59 15.2 mm to (241.2, 124.9), turned to 90 degrees
- moved R15 15.1 mm to (142.6, 133.8), turned to 90 degrees
- moved C102 14.4 mm to (239.4, 128.4), turned to 180 degrees
- moved C105 12.6 mm to (242.6, 136.5), turned to 0 degrees
- moved C90 12.4 mm to (224.4, 138.1), turned to -90 degrees
- moved R18 12.3 mm to (142.6, 135.5), turned to -90 degrees
- moved R58 12.3 mm to (241.4, 127.2), turned to 90 degrees
- moved R12 11.7 mm to (145.3, 147.1)
- moved R13 11.7 mm to (147.0, 147.1)
- moved C14 11.7 mm to (147.2, 134.6), turned to 90 degrees
- moved R11 11.2 mm to (147.0, 145.6)
- moved R10 11.2 mm to (145.3, 145.6)
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Connections:
- C56 pad 2: /HS_MUX/USB_UP2_SSTX_C_P -> /HS_MUX/USB_UP2_SSTX_C_N
- C57 pad 2: /HS_MUX/USB_UP2_SSTX_C_N -> /HS_MUX/USB_UP2_SSTX_C_P
- U11 pad 6: /UPSTREAM_CON1/USB_UP_SSTX_N -> /UPSTREAM_CON1/USB_UP_SSTX_P
- U11 pad 7: /UPSTREAM_CON1/USB_UP_SSTX_P -> /UPSTREAM_CON1/USB_UP_SSTX_N
- U11 pad 8: /UPSTREAM_CON1/USB_UP_SSTX_P -> /UPSTREAM_CON1/USB_UP_SSTX_N
- U11 pad 9: /UPSTREAM_CON1/USB_UP_SSTX_N -> /UPSTREAM_CON1/USB_UP_SSTX_P
- U4 pad 12: /HS_MUX/USB_UP2_SSTX_C_P -> /HS_MUX/USB_UP2_SSTX_C_N
- U4 pad 13: /HS_MUX/USB_UP2_SSTX_C_N -> /HS_MUX/USB_UP2_SSTX_C_P
- U9 pad 6: /UPSTREAM_CON/USB_UP_SSTX_N -> /UPSTREAM_CON/USB_UP_SSTX_P
- U9 pad 7: /UPSTREAM_CON/USB_UP_SSTX_P -> /UPSTREAM_CON/USB_UP_SSTX_N
- U9 pad 8: /UPSTREAM_CON/USB_UP_SSTX_P -> /UPSTREAM_CON/USB_UP_SSTX_N
- U9 pad 9: /UPSTREAM_CON/USB_UP_SSTX_N -> /UPSTREAM_CON/USB_UP_SSTX_P
Routing:
- net /DOWNSTREAM_CONNECTORS/USB_DS_D_N: track 7.75 -> 101.7 mm, vias 0 -> 2
- net /DOWNSTREAM_CONNECTORS/USB_DS_D_P: track 7.75 -> 101.3 mm, vias 0 -> 2
- net /DOWNSTREAM_CONNECTORS1/USB_DS_D_N: track 7.75 -> 71.3 mm, vias 0 -> 2
- net /HS_MUX/USB_UPSW_D_P: track 0.00 -> 63.4 mm, vias 0 -> 2
- net /DOWNSTREAM_CONNECTORS1/USB_DS_D_P: track 7.75 -> 71.0 mm, vias 0 -> 2
- net /HS_MUX/USB_UPSW_D_N: track 0.00 -> 62.2 mm, vias 0 -> 2
- net /UPSTREAM_CON1/USB_UP_D_N: track 12.7 -> 51.4 mm, vias 0 -> 2
- net /UPSTREAM_CON1/USB_UP_D_P: track 13.0 -> 50.9 mm, vias 0 -> 2
- net /DOWNSTREAM_CONNECTORS2/USB_DS_D_N: track 7.75 -> 44.6 mm, vias 0 -> 2
- net /DOWNSTREAM_CONNECTORS2/USB_DS_D_P: track 7.75 -> 43.9 mm, vias 0 -> 2
- net /USB_HUB/USB_UPSW_SSTX_P: track 0.00 -> 30.9 mm, vias 0 -> 2
- net /USB_HUB/USB_UPSW_SSTX_N: track 0.00 -> 30.2 mm, vias 0 -> 2
- net /USB_HUB/USB_UPSW_SSRX_P: track 0.00 -> 29.8 mm, vias 0 -> 2
- net /USB_HUB/USB_UPSW_SSRX_N: track 0.00 -> 28.7 mm, vias 0 -> 2
- net /UPSTREAM_CON/USB_UP_D_P: track 11.6 -> 34.0 mm, vias 0 -> 2
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- added copper zone on B.Cu, net GND
- added copper zone on F.Cu, net GND
- added copper zone on In1.Cu, net GND
- added copper zone on In2.Cu, net GND
- added copper zone on B.Cu, net Net-(J4-VBUS)
- added copper zone on B.Cu, net Net-(J5-VBUS)
- added copper zone on B.Cu, net Net-(J6-VBUS)
- added copper zone on B.Cu, net Net-(J7-VBUS)
- added copper zone on B.Cu, net Net-(U12-OUT)
- added copper zone on B.Cu, net Net-(U14-OUT)
- added copper zone on B.Cu, net Net-(U16-OUT)
- added copper zone on B.Cu, net Net-(U18-OUT)
Other:
- copper layers 6 -> 4

Commit message: Layout + Schematic weiter gemacht
Parts:
- removed R28: R, 00_Resistor:Res_0402
- added C106: 100uF, Capacitor_SMD:CP_Elec_6.3x5.9, F.Cu at (176.2, 113.6)
- added C107: 100uF, Capacitor_SMD:CP_Elec_6.3x5.9, F.Cu at (229.6, 113.6)
- added C108: 100n, 00_Capacitor:Cap_0402, B.Cu at (190.5, 130.7)
- added C109: 100uF, Capacitor_SMD:CP_Elec_6.3x5.9, F.Cu at (228.8, 136.2)
- added C11: 100n, 00_Capacitor:Cap_0402, B.Cu at (152.7, 131.0)
- added C110: 10u, 00_Capacitor:Cap_0603, F.Cu at (237.8, 130.1)
- added C111: 100n, 00_Capacitor:Cap_0402, B.Cu at (237.9, 142.4)
- added C112: 100n, 00_Capacitor:Cap_0402, B.Cu at (244.7, 138.5)
- added C113: 100n, 00_Capacitor:Cap_0402, F.Cu at (248.2, 138.8)
- added C114: 100n, 00_Capacitor:Cap_0402, B.Cu at (240.7, 134.2)
- added D4: BAT54J, Diode_SMD:D_SOD-323F, F.Cu at (237.9, 138.7)
- added D5: BAT54J, Diode_SMD:D_SOD-323F, F.Cu at (238.2, 128.3)
- added D6: MM3Z2V4, Diode_SMD:D_SOD-323F, F.Cu at (240.2, 145.8)
- added Q1: NTJD4401NT1G, Package_TO_SOT_SMD:SOT-363_SC-70-6, F.Cu at (227.4, 128.2)
- added Q2: NTJD4401NT1G, Package_TO_SOT_SMD:SOT-363_SC-70-6, F.Cu at (232.4, 128.2)
- added R60: 10k, 00_Resistor:Res_0402, F.Cu at (251.8, 140.7)
- added R61: 10k, 00_Resistor:Res_0402, F.Cu at (247.8, 137.3)
- added R62: 10k, 00_Resistor:Res_0402, F.Cu at (236.8, 136.3)
- added R63: 100, 00_Resistor:Res_0402, F.Cu at (225.1, 128.9)
- added R64: 10k, 00_Resistor:Res_0402, F.Cu at (235.2, 128.3)
- added R65: 100, 00_Resistor:Res_0402, F.Cu at (229.9, 128.9)
- added R66: 100, 00_Resistor:Res_0402, F.Cu at (235.2, 127.5)
- added R67: 1M, 00_Resistor:Res_0402, F.Cu at (235.2, 129.2)
- added R68: 10k, 00_Resistor:Res_0402, F.Cu at (240.2, 141.8)
- added R69: 10k, 00_Resistor:Res_0402, F.Cu at (240.2, 143.6)
- added R70: 10k, 00_Resistor:Res_0402, F.Cu at (237.3, 145.8)
- added SW1: SW_Omron_B3FS, Button_Switch_SMD:SW_SPST_Omron_B3FS-105xP, F.Cu at (217.1, 131.9)
- added U20: 74LVC1G08, Package_TO_SOT_SMD:SOT-23-5, F.Cu at (240.7, 134.2)
- added U21: 74LVC1G08, Package_TO_SOT_SMD:SOT-23-5, F.Cu at (244.7, 138.5)
- added U22: LM397, Package_TO_SOT_SMD:SOT-23-5, F.Cu at (237.9, 142.4)
- C96, C97: value 10u -> 1u
- D1, D2: value D_Schottky -> BAT54J; footprint Diode_SMD:D_SOD-323 -> Diode_SMD:D_SOD-323F
- H1, H3, H4: footprint MountingHole:MountingHole_3.2mm_M3_DIN965_Pad_TopBottom -> MountingHole:MountingHole_3.2mm_M3_Pad
- H2: footprint MountingHole:MountingHole_3.2mm_M3_Pad_TopBottom -> MountingHole:MountingHole_3.2mm_M3_Pad
- J8: value Conn_01x16_MountingPin -> Conn_01x16_Pin
- J9: value Conn_01x04_MountingPin -> Conn_01x04_Pin
- L1, L2: footprint Inductor_SMD:L_Coilcraft_XAL7030-272 -> Inductor_SMD:L_Wuerth_MAPI-3020
- R15, R16, R18, R19: moved to B.Cu
- R27: value R -> 1k
- R29: value R -> 10k
- U3: footprint Package_SO:VSSOP-10_3x3mm_P0.5mm -> Package_SO:HVSSOP-10-1EP_3x3mm_P0.5mm_EP1.83x1.89mm
- moved H4 121.4 mm to (258.4, 107.2)
- moved H1 113.0 mm to (145.4, 107.2)
- moved H2 47.0 mm to (145.4, 154.2)
- moved C90 32.9 mm to (202.3, 113.6), turned to 90 degrees
- moved L2 20.5 mm to (256.1, 129.0), turned to 90 degrees
- moved C101 17.7 mm to (255.1, 134.8), turned to 90 degrees
- moved C93 17.0 mm to (247.6, 154.2), turned to 0 degrees
- moved R59 16.9 mm to (253.3, 136.8), turned to -90 degrees
- moved C102 16.0 mm to (254.8, 132.4), turned to 90 degrees
- moved C105 15.8 mm to (252.2, 123.9), turned to 180 degrees
- moved C94 15.1 mm to (254.8, 145.9), turned to -90 degrees
- moved R58 14.2 mm to (253.4, 134.7), turned to -90 degrees
- moved L1 13.4 mm to (243.7, 149.3), turned to -90 degrees
- moved C92 13.4 mm to (247.6, 152.3), turned to 0 degrees
- moved C104 13.0 mm to (252.2, 125.9), turned to 180 degrees
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Connections:
- C43 pad 1: Net-(U5-VIN) -> VIN
- J1 pad 1: Net-(U5-VIN) -> VIN
- R27 pad 1: Net-(U5-VIN) -> +5V
- R29 pad 2: Net-(U5-ST) -> unconnected-(R29-Pad2)
- U5 pad 1: Net-(U5-VIN) -> VIN
- U5 pad 5: Net-(U5-ST) -> /POWER_SUPPLY/U5_ST
Routing:
- net +3.3V: track 0.00 -> 16.6 mm, vias 0 -> 12
- net +1V1: track 1.57 -> 13.4 mm, vias 8 -> 13
- net GND: track 12.4 -> 14.7 mm, vias 20 -> 101
- net /POWER_SUPPLY/BUCK_1V1_VCC: track 0.00 -> 1.81 mm
- net Net-(U6-BOOT): track 0.00 -> 1.80 mm
- net Net-(U7-BOOT): track 0.00 -> 1.68 mm
- net /POWER_SUPPLY/BUCK_3V3_VCC: track 0.00 -> 1.61 mm
- net /DOWNSTREAM_CONNECTORS1/USB_DS_D_N: track 71.3 -> 70.0 mm
- net /DOWNSTREAM_CONNECTORS1/USB_DS_D_P: track 71.0 -> 69.6 mm
- net /POWER_SUPPLY/BUCK_3V3_FB: track 0.00 -> 1.31 mm, vias 0 -> 1
- net /DOWNSTREAM_CONNECTORS/USB_DS_D_N: track 101.7 -> 100.4 mm
- net /DOWNSTREAM_CONNECTORS/USB_DS_D_P: track 101.3 -> 100.0 mm
- net /POWER_SUPPLY/BUCK_1V1_FB: track 0.00 -> 1.16 mm, vias 0 -> 1
- net /DOWNSTREAM_CONNECTORS3/~{USB_DS_OC}: track 2.39 -> 1.32 mm
- net /DOWNSTREAM_CONNECTORS2/~{USB_DS_OC}: track 2.51 -> 1.45 mm
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- added copper zone on B.Cu, net +1V1
- added copper zone on F.Cu, net +1V1
- added copper zone on F.Cu, net +3.3V
- added copper zone on B.Cu, net +5V
- added copper zone on F.Cu, net +5V
- added copper zone on F.Cu, net /POWER_SUPPLY/LX_1V1
- added copper zone on F.Cu, net /POWER_SUPPLY/LX_3V3
- added copper zone on B.Cu, net VIN
