File: USB_3_SWITCHER.kicad_pcb (KiCad board)
At the start: 4 copper layers, 122 x 56 mm, 262 parts, among them J1 Jack-DC, J2 Wuerth_USB3_B_Receptable_6922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, J3 Wuerth_USB3_B_Receptable_6922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, J4 Wuerth_USB3_Receptible_692122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, J5 Wuerth_USB3_Receptible_692122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, J6 Wuerth_USB3_Receptible_692122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, J7 Wuerth_USB3_Receptible_692122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, J8 Conn_01x16_Pin, J9 Conn_01x04_Pin, Q1 NTJD4401NT1G, Q2 NTJD4401NT1G, Q3 NTJD4401NT1G, Q4 NTJD4401NT1G, Q5 NTJD4401NT1G, SW1 SW_Omron_B3FS, U1 AT24CS04-SSHM, U10 LM66100DCK, U11 TPD6E05U06RVZ, U12 MAX8586, U13 TPD6E05U06RVZ, U14 MAX8586, U15 TPD6E05U06RVZ, U16 MAX8586, U17 TPD6E05U06RVZ, U18 MAX8586, U19 TPD6E05U06RVZ, U2 TUSB8043A, U20 74LVC1G08, U21 74LVC1G08, U22 LM397, U23 74LVC1G17, U24 74LVC2G74, U25 74LVC1G17, U26 74LVC1G32, U27 74LVC1G08, U28 ISO1540, U3 TS3USB30EDGSR, U4 CBTL02043A, U5 LM66100DCK, U6 LMR33640ADDA, U7 LMR33640ADDA, U8 LM66100DCK, U9 TPD6E05U06RVZ, Y1 24MHz 20ppm

Commit message: Layout nearly finished
Parts:
- added D10: LED, LED_SMD:LED_0603_1608Metric, F.Cu at (241.8, 154.2)
- added D11: LED, LED_THT:LED_D3.0mm_Horizontal_O6.35mm_Z2.0mm, F.Cu at (253.0, 107.0)
- added D12: LED, LED_THT:LED_D3.0mm_Horizontal_O6.35mm_Z2.0mm, F.Cu at (226.5, 107.0)
- added D13: LED, LED_THT:LED_D3.0mm_Horizontal_O6.35mm_Z2.0mm, F.Cu at (200.0, 107.0)
- added D14: LED, LED_THT:LED_D3.0mm_Horizontal_O6.35mm_Z2.0mm, F.Cu at (173.8, 107.0)
- added D3: LED, LED_SMD:LED_0603_1608Metric, F.Cu at (217.0, 127.0)
- added D8: LED, LED_SMD:LED_0603_1608Metric, F.Cu at (217.0, 137.0)
- added D9: LED, LED_SMD:LED_0603_1608Metric, F.Cu at (241.8, 156.8)
- added G***: LOGO, 00_Graphic_Symbols:USB_A_LOGO_1, B.Cu at (183.7, 112.0)
- added G***: LOGO, 00_Graphic_Symbols:USB_A_LOGO_1, B.Cu at (220.8, 146.7)
- added G***: LOGO, 00_Graphic_Symbols:USB_A_LOGO_1, B.Cu at (162.2, 149.5)
- added G***: LOGO, 00_Graphic_Symbols:USB_A_LOGO_1, B.Cu at (236.4, 112.0)
- added G***: LOGO, 00_Graphic_Symbols:ANR_LOGO_F11, B.Cu at (153.8, 120.9)
- added G***: LOGO, 00_Graphic_Symbols:USB_A_LOGO_1, B.Cu at (210.1, 112.0)
- added G***: LOGO, 00_Graphic_Symbols:USB_A_LOGO_1, B.Cu at (157.2, 112.0)
- added Q6: NTJD4401NT1G, Package_TO_SOT_SMD:SOT-363_SC-70-6, F.Cu at (251.7, 110.9)
- added Q7: NTJD4401NT1G, Package_TO_SOT_SMD:SOT-363_SC-70-6, F.Cu at (224.3, 110.7)
- added Q8: NTJD4401NT1G, Package_TO_SOT_SMD:SOT-363_SC-70-6, F.Cu at (197.7, 110.4)
- added Q9: NTJD4401NT1G, Package_TO_SOT_SMD:SOT-363_SC-70-6, F.Cu at (170.9, 111.2)
- added R100: 120, 00_Resistor:Res_0402, F.Cu at (198.2, 113.0)
- added R101: 120, 00_Resistor:Res_0402, F.Cu at (172.6, 109.2)
- added R82: 220, 00_Resistor:Res_0402, F.Cu at (219.8, 126.9)
- added R83: 220, 00_Resistor:Res_0402, F.Cu at (214.9, 137.4)
- added R84: 120, 00_Resistor:Res_0402, F.Cu at (244.2, 156.8)
- added R93: 330, 00_Resistor:Res_0402, F.Cu at (239.8, 152.8)
- added R94: 39k, 00_Resistor:Res_0402, F.Cu at (251.2, 113.5)
- added R95: 39k, 00_Resistor:Res_0402, F.Cu at (224.2, 113.3)
- added R96: 39k, 00_Resistor:Res_0402, F.Cu at (197.2, 113.0)
- added R97: 39k, 00_Resistor:Res_0402, F.Cu at (170.2, 113.8)
- added R98: 120, 00_Resistor:Res_0402, F.Cu at (252.2, 113.5)
- added R99: 120, 00_Resistor:Res_0402, F.Cu at (225.2, 113.3)
- added REF**: LayerMarker_4_6.35x2.54mm_TextH1mm_P1.27mm_BottomMirrored, Symbol:LayerMarker_4_6.35x2.54mm_TextH1mm_P1.27mm_BottomMirrored, F.Cu at (260.9, 120.3)
- added REF**: ESD-Logo_13.2x12mm_SilkScreen, Symbol:ESD-Logo_13.2x12mm_SilkScreen, B.Cu at (236.8, 128.0)
- C118: moved to B.Cu
- moved C127 3.89 mm to (193.5, 135.9), turned to 0 degrees
- moved C118 0.33 mm to (218.8, 136.2)
Routing:
- net +3.3V: track 75.7 -> 189.1 mm, vias 32 -> 44
- net VBUS: track 51.4 -> 115.7 mm
- net /HS_MUX/DIRECTION_SELECT: track 22.3 -> 86.0 mm, vias 3 -> 4
- net /USB_HUB/SMB_SCL: track 36.4 -> 86.5 mm, vias 2 -> 4
- net /USB_HUB/SMB_SDA: track 37.9 -> 85.4 mm, vias 1 -> 3
- net /DIRECTION_SWITCH/DIRECTION: track 23.3 -> 63.0 mm, vias 1 -> 4
- net /HS_MUX/~{MUX_OE}: track 25.1 -> 51.6 mm
- net Net-(D12-A): track 0.00 -> 14.3 mm
- net Net-(D13-A): track 0.00 -> 14.0 mm
- net Net-(D11-A): track 0.00 -> 13.8 mm
- net +5V: track 52.0 -> 60.9 mm
- net /DOWNSTREAM_CONNECTORS/VBUS_OUT_ON: track 134.6 -> 140.8 mm
- net Net-(D14-K): track 0.00 -> 6.02 mm, vias 0 -> 1
- net /DOWNSTREAM_CONNECTORS1/VBUS_OUT_ON: track 104.0 -> 109.5 mm
- net /DIRECTION_SWITCH/~{RESET}: track 167.4 -> 172.8 mm
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- added copper zone on In2.Cu, net +3.3V
Other:
- board text added: "ANR Blastec"
- board text added: "Rev 1"
- board text added: "USB Switcher"

Commit message: Powersequencing
Parts:
- removed D4: BAT54J, Diode_SMD:D_SOD-323F
- removed the REF** at (236.8, 128.0)
- added C129: 100n, 00_Capacitor:Cap_0402, B.Cu at (237.1, 133.8)
- added C130: 100n, 00_Capacitor:Cap_0402, B.Cu at (226.3, 145.9)
- added R102: 10k, 00_Resistor:Res_0402, F.Cu at (244.6, 139.2)
- added R103: 0, 00_Capacitor:Cap_0402, F.Cu at (251.8, 138.9)
- added R104: 10k, 00_Resistor:Res_0402, F.Cu at (227.8, 143.6)
- added U29: 74LVC1G08, Package_TO_SOT_SMD:SOT-23-5, F.Cu at (226.3, 145.9)
- added U30: 74LVC1G08, Package_TO_SOT_SMD:SOT-23-5, F.Cu at (237.1, 133.8)
- C111, R61: moved to F.Cu
- C112, C113: moved to B.Cu
- moved R62 19.2 mm to (244.8, 137.4), turned to 180 degrees
- moved U21 13.4 mm to (241.7, 138.3)
- moved C114 12.8 mm to (241.6, 136.2)
- moved R69 6.20 mm to (237.7, 136.2), turned to 0 degrees
- moved C113 6.02 mm to (232.8, 128.6), turned to -135 degrees
- moved R73 5.60 mm to (242.8, 132.9), turned to 180 degrees
- moved C112 5.48 mm to (242.3, 130.7), turned to -135 degrees
- moved R68 5.48 mm to (236.0, 136.2), turned to 0 degrees
- moved U20 4.58 mm to (232.8, 128.6)
- moved U23 3.89 mm to (242.3, 130.7), turned to 0 degrees
- moved R74 3.81 mm to (237.2, 130.5)
- moved D7 3.77 mm to (237.2, 129.0)
- moved C111 3.70 mm to (233.6, 141.0)
- moved R70 2.98 mm to (235.8, 141.1)
- moved C115 2.92 mm to (239.7, 131.3)
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Connections:
- net /POWER_SUPPLY/BUCK_1V1_PG renamed /POWER_SEQUENCING/BUCK_1V1_PG
- net /POWER_SUPPLY/VREF renamed /POWER_SEQUENCING/VREF
- net /UPSTREAM_CON/USB_UP_PORT_POWER_ON renamed /POWER_SEQUENCING/USB_UP_PORT1_POWER_ON
- net /UPSTREAM_CON1/USB_UP_PORT_POWER_ON renamed /POWER_SEQUENCING/USB_UP_PORT2_POWER_ON
- Q3 pad 2: /POWER_SUPPLY/VIN_PGOOD -> /POWER_SEQUENCING/VIN_PGOOD
- R62 pad 2: Net-(D4-A) -> /POWER_SEQUENCING/VIN_PGOOD
- R72 pad 2: /POWER_SUPPLY/VIN_PGOOD -> /POWER_SEQUENCING/VIN_PGOOD
- U20 pad 1: Net-(U20-Pad1) -> /POWER_SUPPLY/BUCK_3V3_PG
- U21 pad 1: Net-(D4-A) -> Net-(U21-Pad1)
- U21 pad 2: /POWER_SUPPLY/BUCK_3V3_PG -> /POWER_SEQUENCING/VIN_PGOOD
- U21 pad 4: Net-(U20-Pad1) -> /POWER_SEQUENCING/BUCK_3V3_EN
- U22 pad 4: /POWER_SUPPLY/VIN_PGOOD -> /POWER_SEQUENCING/VIN_PGOOD
- U6 pad 3: /POWER_SUPPLY/BUCK_3V3_EN -> /POWER_SEQUENCING/BUCK_3V3_EN
Routing:
- net /POWER_SEQUENCING/USB_UP_PORT2_POWER_ON: track 1.65 -> 69.9 mm, vias 0 -> 2
- net /POWER_SEQUENCING/VIN_PGOOD: track 0.00 -> 44.2 mm
- net /POWER_SUPPLY/VIN_PGOOD: track 40.5 -> 0.00 mm, vias 2 -> 0
- net Net-(R104-Pad2): track 0.00 -> 28.6 mm
- net /HS_MUX/DIRECTION_SELECT: track 86.0 -> 60.6 mm, vias 4 -> 6
- net /POWER_SUPPLY/U5_ST: track 0.00 -> 17.5 mm
- net /POWER_SEQUENCING/BUCK_3V3_EN: track 0.00 -> 14.1 mm, vias 0 -> 2
- net +3.3V: track 189.1 -> 198.8 mm, vias 44 -> 42
- net Net-(D4-A): track 8.61 -> 0.00 mm
- net /DIRECTION_SWITCH/~{RESET}: track 172.8 -> 180.7 mm
- net /DOWNSTREAM_CONNECTORS/~{USB_DS_OC}: track 146.8 -> 139.0 mm
- net /POWER_SUPPLY/BUCK_1V1_EN: track 0.00 -> 6.59 mm
- net Net-(U22-+): track 2.78 -> 9.30 mm
- net /POWER_SUPPLY/BUCK_3V3_PG: track 27.8 -> 33.9 mm
- net /POWER_SEQUENCING/BUCK_1V1_PG: track 14.5 -> 20.2 mm, vias 1 -> 0
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
Commit message: Schaltplan erweitert, Kleinzeug
Parts:
- added C131: 1u, 00_Capacitor:Cap_0402, F.Cu at (226.6, 150.3)
- added C132: 100n, 00_Capacitor:Cap_0402, F.Cu at (248.2, 137.4)
- added R105: 1K, 00_Capacitor:Cap_0402, F.Cu at (245.1, 130.0)
- added SW2: SW_Omron_B3FS, Button_Switch_SMD:SW_SPST_Omron_B3FS-100xP, F.Cu at (152.4, 119.4)
- R32, R35: value R -> 1k
- U29: value 74LVC1G08 -> 74LVC1G32
- moved G*** 22.2 mm to (174.9, 127.8)
Connections:
- R73 pad 1: /DIRECTION_SWITCH/~{RESET} -> Net-(R105-Pad1)
- U23 pad 4: /DIRECTION_SWITCH/~{RESET} -> Net-(R105-Pad1)
Routing:
- net Net-(R105-Pad1): track 0.00 -> 3.40 mm
- net /DIRECTION_SWITCH/~{RESET}: track 180.7 -> 178.9 mm
- net /DOWNSTREAM_CONNECTORS2/VBUS_OUT_ON: track 74.6 -> 75.6 mm
- net /DOWNSTREAM_CONNECTORS3/VBUS_OUT_ON: track 43.7 -> 44.7 mm
