File: DOWNSTREAM_CONNECOTRS.kicad_sch (KiCad schematic)
At the start: 7 parts, among them J6 USB3_A, U11 TPD6E05U06RVZ, U12 MAX8586

Commit message: Arbeit
Parts:
- added C11, C12: 10u, Capacitor_SMD:C_0603_1608Metric, symbol Device:C
- added FB1: FerriteBead, Resistor_SMD:R_0805_2012Metric, symbol Device:FerriteBead
Connections:
- net GND: now also C11.1, C12.2
- net at J6.1 (VBUS): now also C12.1, FB1.2; no longer U12.5 (OUT)
- new net: C11.2, FB1.1, U12.5 (OUT)
Other:
- moved on the sheet: U12

Commit message: Weiter gearbeitet
Fast fertig:
HUB
Fertig
Connector (Up and Down)
MUX
Parts:
- added C13: 1u, Capacitor_SMD:C_0402_1005Metric, symbol Device:C
- added R11, R4, R6, R7: 10k, Resistor_SMD:R_0402_1005Metric, symbol Device:R
- added R3: 39k, Resistor_SMD:R_0402_1005Metric, symbol Device:R
Connections:
- net +5V: now also C13.2, R6.1, R7.1
- net GND: now also C13.1, R3.2
- net at U12.1 (SEL): now also R6.2
- net at U12.2 (ISET): now also R3.1
- net VBUS_OUT_ON: now reaches U12.3 (ON)
- net VBUS_OUT_ON: now also R11.2
- net ~{USB_DS_OC}: now reaches U12.6 (~{FAULT})
- net ~{USB_DS_OC}: now also R4.2
- net at U12.8 (ENRESET): now also R7.2
- new net +3.3V: R11.1, R4.1
Other:
- moved on the sheet: C10, C11, C12, C3, C4, C9, FB1, U11, U12

Commit message: Footprints Updated
Parts:
- C10, C3, C4, C9: footprint (none) -> 00_Capacitor:Cap_0402
- C11, C12: footprint Capacitor_SMD:C_0603_1608Metric -> 00_Capacitor:Cap_0603
- C13: footprint Capacitor_SMD:C_0402_1005Metric -> 00_Capacitor:Cap_0402
- R11, R3, R4, R6, R7: footprint Resistor_SMD:R_0402_1005Metric -> 00_Resistor:Res_0402
Changed lines of the file:
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@@
 			)
 		)
-		(property "Footprint" "Capacitor_SMD:C_0603_1608Metric"
+		(property "Footprint" "00_Capacitor:Cap_0603"
 			(at 176.2252 58.42 0)
 			(effects
@@
 			)
 		)
-		(property "Footprint" ""
+		(property "Footprint" "00_Capacitor:Cap_0402"
 			(at 82.55 92.71 0)
 			(effects
@@
 			)
 		)
-		(property "Footprint" ""
+		(property "Footprint" "00_Capacitor:Cap_0402"
 			(at 88.9 95.25 0)
 			(effects
@@
 			)
 		)
-		(property "Footprint" ""
+		(property "Footprint" "00_Capacitor:Cap_0402"
 			(at 82.55 85.09 0)
 			(effects
@@
 			)
 		)
-		(property "Footprint" "Capacitor_SMD:C_0402_1005Metric"
+		(property "Footprint" "00_Capacitor:Cap_0402"
 			(at 145.0848 34.29 0)
 			(effects
@@
 			)
 		)
-		(property "Footprint" "Resistor_SMD:R_0402_1005Metric"
+		(property "Footprint" "00_Resistor:Res_0402"
 			(at 115.062 54.61 90)
 			(effects
@@
 			)
 		)
-		(property "Footprint" ""
+		(property "Footprint" "00_Capacitor:Cap_0402"
 			(at 88.9 87.63 0)
 			(effects
@@
 			)
 		)
-		(property "Footprint" "Resistor_SMD:R_0402_1005Metric"
+		(property "Footprint" "00_Resistor:Res_0402"
 			(at 115.062 29.21 90)
 			(effects
@@
 			)
 		)
-		(property "Footprint" "Resistor_SMD:R_0402_1005Metric"
+		(property "Footprint" "00_Resistor:Res_0402"
 			(at 69.342 29.21 90)
 			(effects
@@
 			)
 		)
-		(property "Footprint" "Resistor_SMD:R_0402_1005Metric"
+		(property "Footprint" "00_Resistor:Res_0402"
 			(at 106.172 29.21 90)
 			(effects
@@
 			)
 		)
-		(property "Footprint" "Resistor_SMD:R_0402_1005Metric"
+		(property "Footprint" "00_Resistor:Res_0402"
 			(at 96.012 29.21 90)
 			(effects
@@
 			)
 		)
-		(property "Footprint" "Capacitor_SMD:C_0603_1608Metric"
+		(property "Footprint" "00_Capacitor:Cap_0603"
 			(at 159.7152 50.8 0)
 			(effects

Commit message: USB 3 Stecker ausgetauscht
Parts:
- removed J6: USB3_A, symbol Connector:USB3_A
- added J4: Wuerth_USB3_Receptible_692122030100, 00_Connector:Wuerth_USB3A_receptible_692122030100, symbol 00_Connectors_USB:Wuerth_USB3_Receptible_692122030100
- renumbered C3 to C59, C9 to C60, C4 to C61, C10 to C62, C13 to C63, C11 to C64, C12 to C65, R4 to R36, R11 to R37, R7 to R38, R6 to R39, R3 to R40, U11 to U13
Connections:
- net GND: now also J4.4 (GND), J4.7 (GND_DRAIN), J4.S1, J4.S2
- net USB_DS_D_N: now also J4.2 (D-)
- net USB_DS_D_P: now also J4.3 (D+)
- net USB_DS_SSRX_N: now also J4.5 (STDA_SSRX-)
- net USB_DS_SSRX_P: now also J4.6 (STDA_SSRX+)
- net USB_DS_SSTX_N: now also J4.8 (STDA_SSTX-)
- net USB_DS_SSTX_P: now also J4.9 (STDA_SSTX+)
- net at C65.1, FB1.2: now also J4.1 (VBUS)

Commit message: Weiter gemacht
Connections:
- net USB_DS_D_N: now also U13.11 (D2-), U13.4 (NC); no longer U13.1 (NC), U13.14 (D1+)
- net USB_DS_D_P: now also U13.12 (D2+), U13.3 (NC); no longer U13.13 (D1-), U13.2 (NC)
- net USB_DS_SSRX_N: now also U13.1 (NC), U13.14 (D1+); no longer U13.12 (D2+), U13.3 (NC)
- net USB_DS_SSRX_P: now also U13.13 (D1-), U13.2 (NC); no longer U13.11 (D2-), U13.4 (NC)
Other:
- moved on the sheet: U13

Commit message: Layout nearly finished
Parts:
- added D11: LED, LED_THT:LED_D3.0mm_Horizontal_O6.35mm_Z2.0mm, symbol Device:LED
- added Q6: NTJD4401NT1G, Package_TO_SOT_SMD:SOT-363_SC-70-6, symbol ANR_Blastec_Lib:NTJD4401NT1G
- added R94: 39k, 00_Resistor:Res_0402, symbol Device:R
- added R98: 120, 00_Resistor:Res_0402, symbol Device:R
Connections:
- net +3.3V: now also R94.1, R98.2
- net GND: now also Q6.1 (S), Q6.4 (S)
- net VBUS_OUT_ON: now also Q6.2 (G)
- new net: Q6.5 (G), Q6.6 (D), R94.2
- new net: D11.2 (A), R98.1
- new net: D11.1 (K), Q6.3 (D)
