File: POWER_SUPPLY.kicad_sch (KiCad schematic)
At the start: 66 parts, among them J1 Jack-DC, Q1 NTJD4401NT1G, Q2 NTJD4401NT1G, Q3 NTJD4401NT1G, U20 74LVC1G08, U21 74LVC1G08, U22 LM397, U23 74LVC1G17, U5 LM66100DCK, U6 LMR33640ADDA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

Commit message: Layout nearly finished
Parts:
- added D10, D9: LED, LED_SMD:LED_0603_1608Metric, symbol Device:LED
- added R84: 120, 00_Resistor:Res_0402, symbol Device:R
- added R93: 330, 00_Resistor:Res_0402, symbol Device:R
Connections:
- net +3.3V: now also R84.2
- net +5V: now also R93.1
- net GND: now also D10.1 (K), D9.1 (K)
- new net: D10.2 (A), R93.2
- new net: D9.2 (A), R84.1

Commit message: Powersequencing
Parts:
- removed C111, C112, C113, C114: 100n, 00_Capacitor:Cap_0402, symbol Device:C
- removed C115: 1u, 00_Capacitor:Cap_0402, symbol Device:C
- removed D4, D7: BAT54J, Diode_SMD:D_SOD-323F, symbol Diode:BAT54J
- removed D6: MM3Z2V4, Diode_SMD:D_SOD-323F, symbol Diode:MM3Zxx
- removed R61, R62, R68, R69: 10k, 00_Resistor:Res_0402, symbol Device:R
- removed R70: 1k, 00_Resistor:Res_0402, symbol Device:R
- removed R73, R74: 1K, 00_Capacitor:Cap_0402, symbol Device:R
- removed U20, U21: 74LVC1G08, Package_TO_SOT_SMD:SOT-23-5, symbol 74xGxx:74LVC1G08
- removed U22: LM397, Package_TO_SOT_SMD:SOT-23-5, symbol Comparator:LM397
- removed U23: 74LVC1G17, Package_TO_SOT_SMD:SOT-23-5, symbol 74xGxx:74LVC1G17
- added R103: 0, 00_Capacitor:Cap_0402, symbol Device:R
Connections:
- net BUCK_1V1_EN: now also R103.2
- net BUCK_3V3_PG: now also R103.1
- net U5_ST renamed VIN_ST
- no-connect marks 0 -> 2
Other:
- moved on the sheet: C100, C101, C102, C103, C104, C105, C106, C107, C109, C110, C44, C87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

Commit message: Schaltplan erweitert, Kleinzeug
Parts:
- added C132: 100n, 00_Capacitor:Cap_0402, symbol Device:C_Small
Connections:
- net BUCK_3V3_PG: now also C132.2
- net GND: now also C132.1
Other:
- note added: "+5V DC IN max. 4.5A, Polarity Protected"
- note added: "0.5A"
- note added: "0.75A"
- moved on the sheet: C43, J1, R103, R27, R29, U5
