File: UPSTREAM_CON.kicad_sch (KiCad schematic)
At the start: 15 parts, among them J2 Wuerth_USB3_B_Receptable_6922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, U8 LM66100DCK, U9 TPD6E05U06RVZ

Commit message: Powersequencing
Parts:
- R32: now fitted
Changed lines of the file:
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@@
 		(on_board yes)
 		(in_pos_files yes)
-		(dnp yes)
+		(dnp no)
 		(property "Reference" "R32"
 			(at 149.86 54.6099 0)

Commit message: Schaltplan erweitert, Kleinzeug
Parts:
- R32: value R -> 1k
Changed lines of the file:
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@@
 			)
 		)
-		(property "Value" "R"
+		(property "Value" "1k"
 			(at 149.86 57.1499 0)
 			(show_name no)
