File: USB_3_SWITCHER.kicad_sch (KiCad schematic)
At the start: 0 parts

Commit message: Diff Pair neu, Layout fast fertig
Other:
- sheet EXTENSION_HEADER_DEBUG ports: added DIRECTION, DIRECTION_SELECT, SMB_SCL, SMB_SDA, ~{MUX_OE}, ~{RESET}; removed none

Commit message: Powersequencing
Other:
- added sheet POWER_SEQUENCING (POWER_SEQUENCING.kicad_sch)
- sheet POWER_SUPPLY ports: added BUCK_1V1_PG, BUCK_3V3_EN, BUCK_3V3_PG, VIN_PGOOD, VIN_ST; removed ~{RESET}
